File: hackerspacesnl.kicad_pcb (KiCad board)
At the start: 2 copper layers, 129.5 x 159.5 mm, 57 parts, among them J1 Screw_Terminal_01x02, J2 Conn_01x04_Male, Q1 Q_NMOS_GSD, Q2 Q_NMOS_GSD, Q3 Q_NMOS_GSD, Q4 Q_NMOS_GSD, Q5 Q_NMOS_GSD, Q6 Q_NMOS_GSD, SW1 SW_Push, SW2 SW_Push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

Commit message: silkscreen and new gerbers
Routing:
- net GND: track 29.3 -> 28.1 mm
Other:
- board text added: "+5V GND"
Changed lines of the file:
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@@
   (general
     (thickness 1.6)
-    (drawings 5)
-    (tracks 867)
+    (drawings 6)
+    (tracks 865)
     (zones 0)
     (modules 57)
@@
     (add_net led_r4)
   )
+  (module hsnl:LED_0805_multicolor (layer F.Cu)
+    (at 112.5592 54.8937 90)
+    (descr "LED SMD 0805 (2012 Metric), square (rectangular) end terminal, IPC_7351 nominal, (Body size source: https://docs.google.com/spreadsheets/d/1BsfQQcO9C6DZCsRaXUlFlo91Tg2WpOkGARC1WS5S8t0/edit?usp=sharing), generated with kicad-footprint-generator")
+    (tags diode)
+    (attr smd)
+    (fp_text reference D1 (at 0 -1.65 90) (layer F.SilkS) hide
+      (effects (font (size 1 1) (thickness 0.15)))
+    )
+    (fp_text value Red-GreenLED (at 0 1.65 90) (layer F.Fab)
+      (effects (font (size 1 1) (thickness 0.15)))
+    )
+    (fp_text user %R (at 0 0 90) (layer F.Fab)
+      (effects (font (size 0.5 0.5) (thickness 0.08)))
+    )
+    (fp_line (start 1.68 0.95) (end -1.68 0.95) (layer F.CrtYd) (width 0.05))
+    (fp_line (start 1.68 -0.95) (end 1.68 0.95) (layer F.CrtYd) (width 0.05))
+    (fp_line (start -1.68 -0.95) (end 1.68 -0.95) (layer F.CrtYd) (width 0.05))
+    (fp_line (start -1.68 0.95) (end -1.68 -0.95) (layer F.CrtYd) (width 0.05))
+    (fp_line (start -1.685 0.96) (end 1 0.96) (layer F.SilkS) (width 0.12))
+    (fp_line (start -1.685 -0.96) (end -1.685 0.96) (layer F.SilkS) (width 0.12))
+    (fp_line (start 1 -0.96) (end -1.685 -0.96) (layer F.SilkS) (width 0.12))
+    (fp_line (start 1 0.6) (end 1 -0.6) (layer F.Fab) (width 0.1))
+    (fp_line (start -1 0.6) (end 1 0.6) (layer F.Fab) (width 0.1))
+    (fp_line (start -1 -0.3) (end -1 0.6) (layer F.Fab) (width 0.1))
+    (fp_line (start -0.7 -0.6) (end -1 -0.3) (layer F.Fab) (width 0.1))
+    (fp_line (start 1 -0.6) (end -0.7 -0.6) (layer F.Fab) (width 0.1))
+    (pad 3 smd rect (at 0.85 0.525 90) (size 0.9 0.8) (layers F.Cu F.Paste F.Mask)
+      (net 39 "Net-(D1-Pad3)"))
+    (pad 1 smd rect (at -0.85 -0.525 90) (size 0.9 0.8) (layers F.Cu F.Paste F.Mask)
+      (net 40 "Net-(D1-Pad1)"))
+    (pad 4 smd rect (at 0.85 -0.525 90) (size 0.9 0.8) (layers F.Cu F.Paste F.Mask)
+      (net 41 "Net-(D1-Pad4)"))
+    (pad 2 smd rect (at -0.85 0.525 90) (size 0.9 0.8) (layers F.Cu F.Paste F.Mask)
+      (net 42 "Net-(D1-Pad2)"))
+    (model ${KISYS3DMOD}/LED_SMD.3dshapes/LED_0805_2012Metric.wrl
+      (at (xyz 0 0 0))
+      (scale (xyz 1 1 1))
+      (rotate (xyz 0 0 0))
+    )
+  )
   (module hsnl:hsnl (layer F.Cu)
     (at 96.9899 108.6358)
@@
     )
   )
-  (module hsnl:LED_0805_multicolor (layer F.Cu)
-    (at 112.5592 54.8937 90)
-    (descr "LED SMD 0805 (2012 Metric), square (rectangular) end terminal, IPC_7351 nominal, (Body size source: https://docs.google.com/spreadsheets/d/1BsfQQcO9C6DZCsRaXUlFlo91Tg2WpOkGARC1WS5S8t0/edit?usp=sharing), generated with kicad-footprint-generator")
-    (tags diode)
-    (attr smd)
-    (fp_text reference D1 (at 0 -1.65 90) (layer F.SilkS) hide
-      (effects (font (size 1 1) (thickness 0.15)))
-    )
-    (fp_text value Red-GreenLED (at 0 1.65 90) (layer F.Fab)
-      (effects (font (size 1 1) (thickness 0.15)))
-    )
-    (fp_text user %R (at 0 0 90) (layer F.Fab)
-      (effects (font (size 0.5 0.5) (thickness 0.08)))
-    )
-    (fp_line (start 1.68 0.95) (end -1.68 0.95) (layer F.CrtYd) (width 0.05))
-    (fp_line (start 1.68 -0.95) (end 1.68 0.95) (layer F.CrtYd) (width 0.05))
-    (fp_line (start -1.68 -0.95) (end 1.68 -0.95) (layer F.CrtYd) (width 0.05))
-    (fp_line (start -1.68 0.95) (end -1.68 -0.95) (layer F.CrtYd) (width 0.05))
-    (fp_line (start -1.685 0.96) (end 1 0.96) (layer F.SilkS) (width 0.12))
-    (fp_line (start -1.685 -0.96) (end -1.685 0.96) (layer F.SilkS) (width 0.12))
-    (fp_line (start 1 -0.96) (end -1.685 -0.96) (layer F.SilkS) (width 0.12))
-    (fp_line (start 1 0.6) (end 1 -0.6) (layer F.Fab) (width 0.1))
-    (fp_line (start -1 0.6) (end 1 0.6) (layer F.Fab) (width 0.1))
-    (fp_line (start -1 -0.3) (end -1 0.6) (layer F.Fab) (width 0.1))
-    (fp_line (start -0.7 -0.6) (end -1 -0.3) (layer F.Fab) (width 0.1))
-    (fp_line (start 1 -0.6) (end -0.7 -0.6) (layer F.Fab) (width 0.1))
-    (pad 3 smd rect (at 0.85 0.525 90) (size 0.9 0.8) (layers F.Cu F.Paste F.Mask)
-      (net 39 "Net-(D1-Pad3)"))
-    (pad 1 smd rect (at -0.85 -0.525 90) (size 0.9 0.8) (layers F.Cu F.Paste F.Mask)
-      (net 40 "Net-(D1-Pad1)"))
-    (pad 4 smd rect (at 0.85 -0.525 90) (size 0.9 0.8) (layers F.Cu F.Paste F.Mask)
-      (net 41 "Net-(D1-Pad4)"))
-    (pad 2 smd rect (at -0.85 0.525 90) (size 0.9 0.8) (layers F.Cu F.Paste F.Mask)
-      (net 42 "Net-(D1-Pad2)"))
-    (model ${KISYS3DMOD}/LED_SMD.3dshapes/LED_0805_2012Metric.wrl
-      (at (xyz 0 0 0))
-      (scale (xyz 1 1 1))
-      (rotate (xyz 0 0 0))
-    )
-  )
   (module RF_Module:ESP32-WROOM-32 (layer B.Cu)
     (at 48.5197 76.6351 270)
@@
       (effects (font (size 1 1) (thickness 0.15)) (justify mirror))
     )
-    (fp_text value Screw_Terminal_01x02 (at 2.54 -11.2) (layer B.Fab)
+    (fp_text value Screw_Terminal_01x02 (at 2.54 -11.2) (layer B.Fab) hide
       (effects (font (size 1 1) (thickness 0.15)) (justify mirror))
     )
@@
     (fp_line (start 0.95 2) (end 0 0.5) (layer B.Fab) (width 0.1))
     (fp_line (start 0 0.5) (end -0.95 2) (layer B.Fab) (width 0.1))
-    (fp_text user %R (at 2.54 1.3) (layer B.Fab)
+    (fp_text user %R (at 2.54 1.3) (layer B.Fab) hide
       (effects (font (size 1 1) (thickness 0.15)) (justify mirror))
     )
@@
     )
   )
+  (gr_text "+5V\nGND" (at 145.034 144.3482 270) (layer B.SilkS)
+    (effects (font (size 3 2) (thickness 0.15)) (justify mirror))
+  )
   (gr_text "hoera10jaar 2020-01-25\nCC-BY-NC\nStichting Revelation Space\nHackerspace Den Haag\nMakerspace Leidschendam" (at 120.08104 176.19472) (layer B.SilkS)
     (effects (font (size 2 2) (thickness 0.15)) (justify left mirror))
@@
   (segment (start 141.67084 148.7803) (end 142.62862 149.73808) (width 1) (layer F.Cu) (net 1))
   (segment (start 141.67084 140.49756) (end 141.67084 148.7803) (width 1) (layer F.Cu) (net 1))
-  (segment (start 144.66862 149.73808) (end 142.62862 149.73808) (width 1) (layer F.Cu) (net 1))
-  (segment (start 145.4404 148.9663) (end 144.66862 149.73808) (width 1) (layer F.Cu) (net 1))
-  (segment (start 145.4404 140.48232) (end 145.4404 148.9663) (width 1) (layer F.Cu) (net 1))
   (via (at 40.69588 65.3796) (size 0.8) (drill 0.4) (layers F.Cu B.Cu) (net 1))
   (via (at 39.9796 74.38136) (size 0.8) (drill 0.4) (layers F.Cu B.Cu) (net 1))
@@
   (via (at 126.47676 153.60396) (size 0.8) (drill 0.4) (layers F.Cu B.Cu) (net 1))
   (via (at 89.81948 117.68836) (size 0.8) (drill 0.4) (layers F.Cu B.Cu) (net 1))
+  (segment (start 145.4404 146.9263) (end 142.62862 149.73808) (width 1) (layer F.Cu) (net 1))
+  (segment (start 145.4404 140.48232) (end 145.4404 146.9263) (width 1) (layer F.Cu) (net 1))
   (segment (start 147.00016 135.09936) (end 147.00016 138.59256) (width 1) (layer F.Cu) (net 2))
   (segment (start 146.4958 134.595) (end 147.00016 135.09936) (width 1) (layer F.Cu) (net 2))
   (segment (start 147.0154 138.6078) (end 147.00016 138.59256) (width 1) (layer F.Cu) (net 2))
   (segment (start 147.0154 140.48232) (end 147.0154 138.6078) (width 1) (layer F.Cu) (net 2))
-  (segment (start 147.0154 143.63212) (end 147.84324 144.45996) (width 1) (layer F.Cu) (net 2))
-  (segment (start 147.0154 140.48232) (end 147.0154 143.63212) (width 1) (layer F.Cu) (net 2))
+  (segment (start 147.0154 143.90136) (end 147.70862 144.59458) (width 1) (layer F.Cu) (net 2))
   (segment (start 147.70862 144.59458) (end 147.70862 149.73808) (width 1) (layer F.Cu) (net 2))
-  (segment (start 147.84324 144.45996) (end 147.70862 144.59458) (width 1) (layer F.Cu) (net 2))
+  (segment (start 147.0154 140.48232) (end 147.0154 143.90136) (width 1) (layer F.Cu) (net 2))
   (segment (start 144.1958 137.7038) (end 144.1958 134.595) (width 1) (layer F.Cu) (net 3))
   (segment (start 143.3426 138.557) (end 144.1958 137.7038) (width 1) (layer F.Cu) (net 3))

Commit message: versie zoals besteld
Parts:
- moved Ref** 6.89 mm to (131.1, 173.2)

Commit message: nieuwe rev
Connections:
- U2 pad 11: Net-(U2-Pad11) -> led_r1
- U2 pad 12: Net-(U2-Pad12) -> led_r0
- U2 pad 6: led_r0 -> Net-(U2-Pad6)
- U2 pad 7: led_r1 -> Net-(U2-Pad7)
Routing:
- net led_r4: track 56.2 -> 70.8 mm, vias 4 -> 2
- net led_r0: track 36.3 -> 28.2 mm, vias 1 -> 3
- net led_r1: track 43.7 -> 36.3 mm, vias 2 -> 4
- net led_r3: track 62.3 -> 66.3 mm
- net Net-(D12-Pad3): track 102.9 -> 100.9 mm
- net Net-(D10-Pad2): track 104.4 -> 103.1 mm
- net led_r2: track 58.5 -> 59.7 mm
- net Net-(D12-Pad4): track 96.3 -> 95.6 mm
- net Net-(D1-Pad2): track 143.2 -> 142.5 mm
- net Net-(D14-Pad4): track 97.1 -> 97.8 mm
Other:
- board text added: "2009: RandomData (Utrecht) 2009: RevSpace (Den Haag) 2010: Hack42 (Arnhem) 2010-2017: Sk1llz (Almere) 2010: ACKspace (Heerlen) 2011: TkkrLab (Enschede) 2011: Bitlair (Amersfoort) 2011: Frack (Leeuwarden) 2011: TechInc (Amsterdam) 2012: NURDspace (Wageningen) 2014: TDvenlo (Venlo dus) 2014: Bhack (Zwolle) 2015: Pixelbar (Rotterdam) 2018: Hackerspace Nijmegen (Nijmegen dus) 2018: Hackalot (Eindhove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"
- board text removed: "2009: RandomData (Utrecht) 2009: RevSpace (Den Haag) 2010: Hack42 (Arnhem) 2010-2017: Sk1llz (Almere) 2010: ACKspace (Heerlen) 2011: TkkrLab (Enschede) 2011: Bitlair (Amersfoort) 2011: Frack (Leeuwarden) 2011: TechInc (Amsterdam) 2012: NURDspace (Wageningen) 2014: TDvenlo (Venlo dus) 2015: Pixelbar (Rotterdam) 2018: Hackerspace Nijmegen (Nijmegen dus) 2018: Hackalot (Eindhoven)"
