File: hackerspacesnl.sch (KiCad schematic (older format))
At the start: 55 parts, among them J1 Screw_Terminal_01x02, J2 Conn_01x04_Male, Q1 Q_NMOS_GSD, Q2 Q_NMOS_GSD, Q3 Q_NMOS_GSD, Q4 Q_NMOS_GSD, Q5 Q_NMOS_GSD, Q6 Q_NMOS_GSD, SW1 SW_Push, SW2 SW_Push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

Commit message: halverwege component plaatsing
Parts:
- gave numbers to parts that had none: 3
Connections:
- wire segments 192 -> 184
Changed lines of the file:
@@
 	1    0    0    -1
 $EndComp
-Text GLabel 7800 4400 3    50   Input ~ 0
+Text GLabel 10200 4550 2    50   Input ~ 0
 led_r1
-Text GLabel 8850 4500 3    50   Input ~ 0
+Text GLabel 10200 4700 2    50   Input ~ 0
 led_r2
-Text GLabel 9000 4500 3    50   Input ~ 0
+Text GLabel 10200 4850 2    50   Input ~ 0
 led_r3
-Text GLabel 9100 3850 2    50   Input ~ 0
+Text GLabel 10200 5000 2    50   Input ~ 0
 led_r4
-Text GLabel 9100 2850 2    50   Input ~ 0
+Text GLabel 10600 4400 2    50   Input ~ 0
 led_c0
-Text GLabel 9100 3150 2    50   Input ~ 0
+Text GLabel 10600 4550 2    50   Input ~ 0
 led_c1
-Text GLabel 9100 3350 2    50   Input ~ 0
+Text GLabel 10600 4700 2    50   Input ~ 0
 led_c2
-Text GLabel 9100 3450 2    50   Input ~ 0
+Text GLabel 10600 4850 2    50   Input ~ 0
 led_c3
-Text GLabel 9100 3550 2    50   Input ~ 0
+Text GLabel 10600 5000 2    50   Input ~ 0
 led_c4
-Text GLabel 9100 3650 2    50   Input ~ 0
+Text GLabel 10600 5150 2    50   Input ~ 0
 led_c5
 NoConn ~ 7350 2950
@@
 Wire Wire Line
 	9600 3500 9600 3550
-Wire Wire Line
-	9100 2850 8900 2850
-Wire Wire Line
-	9100 3150 8900 3150
-Wire Wire Line
-	9100 3350 8900 3350
-Wire Wire Line
-	8900 3450 9100 3450
-Wire Wire Line
-	9100 3550 8900 3550
-Wire Wire Line
-	8900 3650 9100 3650
-Wire Wire Line
-	9100 3850 8900 3850
-Wire Wire Line
-	7800 4400 7800 4250
-Text GLabel 7050 3650 0    50   Input ~ 0
+Text GLabel 10200 4400 2    50   Input ~ 0
 led_r0
 $Comp
-L Device:R R?
+L Device:R R19
 U 1 1 5E08F19E
 P 7250 4100
-F 0 "R?" H 7320 4146 50  0000 L CNN
+F 0 "R19" H 7320 4146 50  0000 L CNN
 F 1 "10K" H 7320 4055 50  0000 L CNN
 F 2 "Resistor_SMD:R_0603_1608Metric" V 7180 4100 50  0001 C CNN
@@
 $EndComp
 $Comp
-L power:GND #PWR?
+L power:GND #PWR0101
 U 1 1 5E08FA41
 P 7250 4350
-F 0 "#PWR?" H 7250 4100 50  0001 C CNN
+F 0 "#PWR0101" H 7250 4100 50  0001 C CNN
 F 1 "GND" H 7255 4177 50  0000 C CNN
 F 2 "" H 7250 4350 50  0001 C CNN
@@
 	7250 3850 7350 3850
 $Comp
-L Device:R R?
+L Device:R R21
 U 1 1 5E0D9D1B
 P 8600 4500
-F 0 "R?" H 8670 4546 50  0000 L CNN
+F 0 "R21" H 8670 4546 50  0000 L CNN
 F 1 "10K" H 8670 4455 50  0000 L CNN
 F 2 "Resistor_SMD:R_0603_1608Metric" V 8530 4500 50  0001 C CNN
@@
 $EndComp
 $Comp
-L Device:R R?
+L Device:R R20
 U 1 1 5E0DA0FC
 P 8500 4500
-F 0 "R?" H 8570 4546 50  0000 L CNN
+F 0 "R20" H 8570 4546 50  0000 L CNN
 F 1 "10K" H 8570 4455 50  0000 L CNN
 F 2 "Resistor_SMD:R_0603_1608Metric" V 8430 4500 50  0001 C CNN
@@
 $EndComp
 $Comp
-L power:GND #PWR?
+L power:GND #PWR0102
 U 1 1 5E0DA27C
 P 8600 4750
-F 0 "#PWR?" H 8600 4500 50  0001 C CNN
+F 0 "#PWR0102" H 8600 4500 50  0001 C CNN
 F 1 "GND" H 8605 4577 50  0000 C CNN
 F 2 "" H 8600 4750 50  0001 C CNN

Commit message: update
Parts:
- removed C7: 100nF, Capacitor_SMD:C_0603_1608Metric, symbol Device:C
Changed lines of the file:
@@
-$EndComp
-$Comp
-L Device:C C7
-U 1 1 5DFB3FF5
-P 7450 1450
-F 0 "C7" H 7565 1496 50  0000 L CNN
-F 1 "100nF" H 7565 1405 50  0000 L CNN
-F 2 "Capacitor_SMD:C_0603_1608Metric" H 7488 1300 50  0001 C CNN
-F 3 "~" H 7450 1450 50  0001 C CNN
-	1    7450 1450
-	1    0    0    -1
 $EndComp
 $Comp
@@
 F 3 "" H 6950 2350 50  0001 C CNN
 	1    6950 2350
-	1    0    0    -1
-$EndComp
-$Comp
-L power:+3.3V #PWR018
-U 1 1 5DFB8264
-P 7450 1300
-F 0 "#PWR018" H 7450 1150 50  0001 C CNN
-F 1 "+3.3V" H 7465 1473 50  0000 C CNN
-F 2 "" H 7450 1300 50  0001 C CNN
-F 3 "" H 7450 1300 50  0001 C CNN
-	1    7450 1300
 	1    0    0    -1
 $EndComp
@@
 	5850 2700 5850 2800
 $Comp
-L power:GND #PWR019
-U 1 1 5DFE9662
-P 7450 1600
-F 0 "#PWR019" H 7450 1350 50  0001 C CNN
-F 1 "GND" H 7455 1427 50  0000 C CNN
-F 2 "" H 7450 1600 50  0001 C CNN
-F 3 "" H 7450 1600 50  0001 C CNN
-	1    7450 1600
-	1    0    0    -1
-$EndComp
-$Comp
 L power:GND #PWR014

Commit message: layout almost done
Parts:
- removed R19, R20, R21: 10K, Resistor_SMD:R_0603_1608Metric, symbol Device:R
- C1: LCSC (none) -> C19702
- C2, C3, C4, C5: LCSC (none) -> C14663
- C6: LCSC (none) -> C108053
- D1, D10, D11, D12, D13, D14, D15, D2, D3, D5, D6, D7, D8, D9: LCSC (none) -> C391863
- D4: value Red-GreenLED-parts -> Red-GreenLED; LCSC (none) -> C391863
- Q1, Q2, Q3, Q4, Q5, Q6: LCSC (none) -> C181087
- R1, R3, R5, R7, R9: LCSC (none) -> C22828
- R10, R11, R12, R13, R14, R15, R16, R2, R4, R6, R8: LCSC (none) -> C25199
- R17, R18: LCSC (none) -> C25804
- U1: LCSC (none) -> C351784
Connections:
- wire segments 184 -> 191
- no-connect marks 3 -> 6

Commit message: versie zoals besteld
Parts:
- C6: LCSC C108053 -> C16780
- U1: LCSC C351784 -> C6186
Changed lines of the file:
@@
 F 2 "Package_TO_SOT_SMD:SOT-223-3_TabPin2" H 5850 5100 50  0001 C CNN
 F 3 "http://www.advanced-monolithic.com/pdf/ds1117.pdf" H 5950 4650 50  0001 C CNN
-F 4 "C351784" H 5850 4900 50  0001 C CNN "LCSC"
+F 4 "C6186" H 5850 4900 50  0001 C CNN "LCSC"
 	1    5850 4900
 	1    0    0    -1
@@
 F 2 "Capacitor_SMD:C_0805_2012Metric" H 7038 4900 50  0001 C CNN
 F 3 "~" H 7000 5050 50  0001 C CNN
-F 4 "C108053" H 7000 5050 50  0001 C CNN "LCSC"
+F 4 "C16780" H 7000 5050 50  0001 C CNN "LCSC"
 	1    7000 5050
 	1    0    0    -1

Commit message: nieuwe rev
Changed lines of the file:
@@
 	1    0    0    -1
 $EndComp
-Text GLabel 7250 3150 0    50   Input ~ 0
+Text GLabel 7250 3550 0    50   Input ~ 0
 led_r1
 Text GLabel 7250 3250 0    50   Input ~ 0
@@
 Wire Wire Line
 	9600 3500 9600 3550
-Text GLabel 7250 3050 0    50   Input ~ 0
+Text GLabel 7250 3650 0    50   Input ~ 0
 led_r0
 Wire Wire Line
@@
 	9000 3150 8900 3150
 Wire Wire Line
-	7350 3050 7250 3050
-Wire Wire Line
-	7250 3150 7350 3150
-Wire Wire Line
 	7350 3250 7250 3250
 Wire Wire Line
@@
 Wire Wire Line
 	8900 3850 9100 3850
+Wire Wire Line
+	7250 3550 7350 3550
+Wire Wire Line
+	7350 3650 7250 3650
 $EndSCHEMATC
